File: pcb/CDR/_autosave-pcb.kicad_pcb (KiCad board)
At the start: 2 copper layers, 52 x 65.9 mm, 56 parts, among them J1 Conn_01x03_Male, J10 V Reg in, J11 V reg out, J12 V Solar, J13 V batt, J14 V chrg out, J15 V Low Batt in, J16 V ref in, J17 V Batt in, J18 V Low Batt out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

Commit message: Merge branch 'main' of http://github.com/dgibb/sdp into main
Parts:
- removed J11: V reg out, Connector_PinHeader_2.54mm:PinHeader_1x02_P2.54mm_Vertical
- removed J15: V Low Batt in, Connector_PinHeader_2.54mm:PinHeader_1x02_P2.54mm_Vertical
- removed J18: V Low Batt out, Connector_PinHeader_2.54mm:PinHeader_1x02_P2.54mm_Vertical
- removed J7: V sys in, Connector_PinHeader_2.54mm:PinHeader_1x02_P2.54mm_Vertical
- L1: footprint Inductor_SMD:L_1206_3216Metric -> Inductor_SMD:L_Bourns-SRU8028_8.0x8.0mm
- U4: footprint Package_SO:SOIC-8_3.9x4.9mm_P1.27mm -> Package_DIP:DIP-8_W7.62mm
- moved L1 39.6 mm to (99.2, 122.3)
- moved R7 22.2 mm to (109.7, 108.8), turned to -90 degrees
- moved J17 21.7 mm to (115.6, 108.3), turned to -90 degrees
- moved J16 17.2 mm to (98.4, 103.4)
- moved R6 14.2 mm to (114.3, 111.4)
- moved C13 7.41 mm to (118.9, 109.3), turned to 90 degrees
- moved U4 7.35 mm to (109.9, 115.8)
- moved R9 5.44 mm to (128.9, 122.3), turned to 0 degrees
- moved R11 4.72 mm to (121.8, 109.6)
Connections:
- U3 pad EPAD: GND -> (no net)
- U4 pad 2: Net-(J16-Pad1) -> Net-(R6-Pad2)
- U4 pad 3: Net-(R6-Pad2) -> Net-(J16-Pad1)
- Y1 pad 2: GND -> Net-(C5-Pad2)
- Y1 pad 3: Net-(C5-Pad2) -> (no net)
- Y1 pad 4: GND -> (no net)
Routing:
- net Net-(J17-Pad1): track 28.0 -> 3.15 mm
- net Net-(J16-Pad1): track 13.4 -> 0.00 mm
- net Net-(C11-Pad1): track 10.0 -> 0.00 mm
- net VCC: track 98.5 -> 89.5 mm
- net Net-(J15-Pad1): track 7.16 -> 0.00 mm
- net Net-(C7-Pad1): track 23.5 -> 30.2 mm
- net Net-(D7-Pad1): track 8.17 -> 12.2 mm
- net Net-(D7-Pad2): track 10.4 -> 8.87 mm
