File: pcb/CDR/pcb.kicad_pcb (KiCad board)
At the start: 2 copper layers, 13 parts, among them J1 Conn_01x03_Male, J2 Conn_01x03_Male, J3 Conn_01x03_Male, J4 Conn_01x03_Male, J5 Conn_01x04_Female, J6 Conn_01x08_Female, J7 Conn_01x02_Female, U1 ATmega328-P, Y1 16MHz

Commit message: cdr pcb
Parts:
- added C10: 10uF, Capacitor_SMD:C_1206_3216Metric, F.Cu at (128.3, 104.0)
- added C11: 10uF, Capacitor_SMD:C_1206_3216Metric, F.Cu at (123.3, 125.1)
- added C12: 10uF, Capacitor_SMD:C_1206_3216Metric, F.Cu at (153.3, 91.3)
- added C3: 0.1uF, Capacitor_SMD:C_1206_3216Metric, F.Cu at (148.4, 108.0)
- added C6: 22uF, Capacitor_SMD:C_1206_3216Metric, F.Cu at (138.0, 133.1)
- added C7: 220uF, Capacitor_SMD:C_1206_3216Metric, F.Cu at (145.3, 130.7)
- added C8: 10uF, Capacitor_SMD:C_1206_3216Metric, F.Cu at (117.8, 85.3)
- added C9: 1uF, Capacitor_SMD:C_1206_3216Metric, F.Cu at (124.2, 88.3)
- added D1: Red, Diode_SMD:D_1206_3216Metric, F.Cu at (116.0, 102.0)
- added D2: Green, Diode_SMD:D_1206_3216Metric, F.Cu at (112.0, 101.7)
- added D3: CMPSH3-40MA, Diode_SMD:D_SMB, F.Cu at (126.0, 82.2)
- added D4: CMPSH1-4, Diode_SMD:D_SMA, F.Cu at (124.2, 95.1)
- added D5: CMPSH3-40MA, Diode_SMD:D_SMB, F.Cu at (110.9, 88.5)
- added D6: 11DQ06, Diode_SMD:D_SMA, F.Cu at (151.7, 122.8)
- added D7: 1V, Diode_SMD:D_SOD-123, F.Cu at (123.4, 118.1)
- added J10: V Reg in, Connector_PinHeader_2.54mm:PinHeader_1x02_P2.54mm_Vertical, F.Cu at (140.0, 136.1)
- added J11: V reg out, Connector_PinHeader_2.54mm:PinHeader_1x02_P2.54mm_Vertical, F.Cu at (146.3, 125.4)
- added J12: V Solar, Connector_PinHeader_2.54mm:PinHeader_1x02_P2.54mm_Vertical, F.Cu at (112.9, 80.3)
- added J13: V batt, Connector_PinHeader_2.54mm:PinHeader_1x02_P2.54mm_Vertical, F.Cu at (123.5, 101.9)
- added J14: V chrg out, Connector_PinHeader_2.54mm:PinHeader_1x02_P2.54mm_Vertical, F.Cu at (119.4, 102.0)
- added J15: V Low Batt in, Connector_PinHeader_2.54mm:PinHeader_1x02_P2.54mm_Vertical, F.Cu at (131.7, 122.1)
- added J16: V ref in, Connector_PinHeader_2.54mm:PinHeader_1x02_P2.54mm_Vertical, F.Cu at (112.6, 125.9)
- added J17: V Batt in, Connector_PinHeader_2.54mm:PinHeader_1x02_P2.54mm_Vertical, F.Cu at (110.2, 115.1)
- added J18: V Low Batt out, Connector_PinHeader_2.54mm:PinHeader_1x02_P2.54mm_Vertical, F.Cu at (118.0, 128.7)
- added J8: Cell Module, Connector_PinHeader_2.54mm:PinHeader_1x02_P2.54mm_Vertical, F.Cu at (132.2, 115.5)
- added J9: V reg out, Connector_PinHeader_2.54mm:PinHeader_1x02_P2.54mm_Vertical, F.Cu at (151.7, 131.2)
- added L1: 330 uH, Inductor_SMD:L_1206_3216Metric, F.Cu at (138.1, 129.8)
- added L2: 10uH, Inductor_SMD:L_1206_3216Metric, F.Cu at (127.9, 88.6)
- added R1: 1K, Resistor_SMD:R_1206_3216Metric, F.Cu at (145.2, 135.9)
- added R10: 0/160, Resistor_SMD:R_1206_3216Metric, F.Cu at (147.6, 91.1)
- added R2: 3.1k, Resistor_SMD:R_1206_3216Metric, F.Cu at (145.3, 133.3)
- added R3: 5.1k, Resistor_SMD:R_1206_3216Metric, F.Cu at (116.1, 95.7)
- added R4: 5.1k, Resistor_SMD:R_1206_3216Metric, F.Cu at (112.2, 95.6)
- added R5: 0.05, Resistor_SMD:R_1206_3216Metric, F.Cu at (127.8, 95.3)
- added R6: 100k, Resistor_SMD:R_1206_3216Metric, F.Cu at (114.7, 115.9)
- added R7: 220k, Resistor_SMD:R_1206_3216Metric, F.Cu at (114.7, 111.8)
- added R8: 50k, Resistor_SMD:R_1206_3216Metric, F.Cu at (128.6, 117.3)
- added R9: 160, Resistor_SMD:R_1206_3216Metric, F.Cu at (123.5, 122.1)
- added U2: LM2574HVM-12, Package_SO:SOIC-14W_7.5x9mm_P1.27mm, F.Cu at (128.1, 132.8)
- added U3: LT3650EMSE-8.4-PBF, footprints:LT3650EMSE-8.4-PBF, F.Cu at (118.8, 90.3)
- added U4: LM311, Package_SO:SOIC-8_3.9x4.9mm_P1.27mm, F.Cu at (115.1, 121.0)
- J6: value Conn_01x08_Female -> SD Card Reader; footprint Connector_PinSocket_2.54mm:PinSocket_1x08_P2.54mm_Vertical -> Connector_PinHeader_2.54mm:PinHeader_1x06_P2.54mm_Vertical
- J7: value Conn_01x02_Female -> V sys in
- Y1: footprint Crystal:Crystal_SMD_3225-4Pin_3.2x2.5mm -> Crystal:Crystal_SMD_TXC_7M-4Pin_3.2x2.5mm
- moved J7 39.0 mm to (138.9, 125.6)
- moved J6 31.1 mm to (131.5, 100.2), turned to 180 degrees
- moved J1 24.0 mm to (147.8, 119.3), turned to 180 degrees
- moved Y1 19.5 mm to (131.9, 110.0), turned to 180 degrees
- moved J2 15.7 mm to (152.8, 102.1)
- moved U1 14.7 mm to (135.9, 87.5)
- moved C1 14.6 mm to (132.4, 105.2)
- moved J3 14.5 mm to (153.1, 95.1)
- moved C2 14.4 mm to (148.4, 105.4)
- moved C4 14.2 mm to (126.7, 108.3), turned to 0 degrees
- moved J4 13.4 mm to (153.0, 87.8)
- moved C5 10.9 mm to (126.5, 112.5), turned to 0 degrees
- moved J5 3.80 mm to (135.8, 78.5)
Connections:
- J6 pad 1: Net-(J6-Pad1) -> GND
- J6 pad 2: Net-(J6-Pad2) -> VCC
- U1 pad 11: Net-(J6-Pad6) -> unconnected-(U1-Pad11)
- U1 pad 12: Net-(J6-Pad7) -> Net-(J8-Pad1)
- U1 pad 13: Net-(J6-Pad8) -> Net-(J8-Pad2)
- U1 pad 14: unconnected-(U1-Pad14) -> Net-(J15-Pad1)
- U1 pad 2: Net-(J6-Pad1) -> Net-(J6-Pad6)
- U1 pad 26: Net-(J4-Pad3) -> Net-(C12-Pad2)
- U1 pad 3: Net-(J6-Pad2) -> Net-(J6-Pad5)
- U1 pad 4: Net-(J6-Pad3) -> Net-(J6-Pad4)
- U1 pad 5: Net-(J6-Pad4) -> Net-(J6-Pad3)
- U1 pad 6: Net-(J6-Pad5) -> unconnected-(U1-Pad6)
- Y1 pad 2: Net-(C5-Pad2) -> GND
- Y1 pad 3: (no net) -> Net-(C5-Pad2)
- Y1 pad 4: (no net) -> GND
Routing:
- net VCC: track 33.2 -> 98.5 mm
- net Net-(C8-Pad1): track 0.00 -> 42.0 mm
- net Net-(R1-Pad2): track 0.00 -> 35.6 mm
- net Net-(C10-Pad1): track 0.00 -> 30.1 mm
- net Net-(D6-Pad1): track 0.00 -> 25.1 mm, vias 0 -> 2
- net Net-(C7-Pad1): track 0.00 -> 23.5 mm
- net Net-(J17-Pad1): track 0.00 -> 18.3 mm
- net Net-(J6-Pad1): track 17.4 -> 0.00 mm
- net Net-(J6-Pad2): track 17.4 -> 0.00 mm
- net Net-(R6-Pad2): track 0.00 -> 17.2 mm
- net Net-(C9-Pad1): track 0.00 -> 16.2 mm
- net GND: track 21.1 -> 6.27 mm, vias 0 -> 10
- net Net-(J6-Pad5): track 17.4 -> 4.79 mm
- net Net-(J6-Pad4): track 17.4 -> 4.79 mm
- net Net-(J6-Pad3): track 17.4 -> 4.79 mm
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- added copper zone on B.Cu, net GND
- added copper zone on F.Cu, net GND
Other:
- board outline added: 52 x 65.9 mm

Commit message: pcb and analytics updates
Parts:
- moved R7 19.8 mm to (110.1, 131.0), turned to 90 degrees
- moved J17 15.3 mm to (114.2, 129.9), turned to 0 degrees
- moved J16 10.9 mm to (113.4, 115.0), turned to 90 degrees
- moved R6 9.83 mm to (112.8, 125.5)
- moved J10 2.62 mm to (137.4, 136.3), turned to 90 degrees
- moved J12 2.50 mm to (110.4, 80.3), turned to 90 degrees
- moved J15 2.21 mm to (131.4, 124.3)
- moved J18 1.20 mm to (119.2, 128.7)
- moved C11 0.30 mm to (123.3, 125.4)
- turned U4 to 0 degrees
Connections:
- U3 pad EPAD: (no net) -> GND
Routing:
- net Net-(D5-Pad2): track 0.00 -> 6.27 mm
- net GND: track 6.27 -> 0.00 mm, vias 10 -> 20
- net Net-(D7-Pad1): track 11.4 -> 5.59 mm
- net Net-(R6-Pad2): track 17.2 -> 11.8 mm
- net Net-(J15-Pad1): track 4.86 -> 7.16 mm
- net Net-(J17-Pad1): track 18.3 -> 16.1 mm
- net Net-(J16-Pad1): track 11.7 -> 11.0 mm
- net Net-(R3-Pad2): track 4.81 -> 5.33 mm

Commit message: decoupling cap on lm 311
Parts:
- added C13: 1uF, Capacitor_SMD:C_1206_3216Metric, F.Cu at (116.2, 116.2)
- moved J16 2.61 mm to (113.1, 112.4)
Routing:
- net Net-(J17-Pad1): track 16.1 -> 20.5 mm
- net Net-(J16-Pad1): track 11.0 -> 13.4 mm
Changed lines of the file:
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@@
+    )
+  )
+  (footprint "Capacitor_SMD:C_1206_3216Metric" (layer "F.Cu")
+    (at 116.2 116.2)
+    (descr "Capacitor SMD 1206 (3216 Metric), square (rectangular) end terminal, IPC_7351 nominal, (Body size source: IPC-SM-782 page 76, https://www.pcb-3d.com/wordpress/wp-content/uploads/ipc-sm-782a_amendment_1_and_2.pdf), generated with kicad-footprint-generator")
+    (tags "capacitor")
+    (property "Sheetfile" "pcb.kicad_sch")
+    (property "Sheetname" "")
+    (attr smd)
+    (fp_text reference "C13" (at 3 -1.6) (layer "F.SilkS")
+      (effects (font (size 1 1) (thickness 0.15)))
+    )
+    (fp_text value "1uF" (at 0 1.85) (layer "F.Fab")
+      (effects (font (size 1 1) (thickness 0.15)))
+    )
+    (fp_text user "${REFERENCE}" (at 0 0) (layer "F.Fab")
+      (effects (font (size 0.8 0.8) (thickness 0.12)))
+    )
+    (fp_line (start -0.711252 -0.91) (end 0.711252 -0.91) (layer "F.SilkS") (width 0.12))
+    (fp_line (start -0.711252 0.91) (end 0.711252 0.91) (layer "F.SilkS") (width 0.12))
+    (fp_line (start 2.3 1.15) (end -2.3 1.15) (layer "F.CrtYd") (width 0.05))
+    (fp_line (start -2.3 1.15) (end -2.3 -1.15) (layer "F.CrtYd") (width 0.05))
+    (fp_line (start -2.3 -1.15) (end 2.3 -1.15) (layer "F.CrtYd") (width 0.05))
+    (fp_line (start 2.3 -1.15) (end 2.3 1.15) (layer "F.CrtYd") (width 0.05))
+    (fp_line (start 1.6 0.8) (end -1.6 0.8) (layer "F.Fab") (width 0.1))
+    (fp_line (start 1.6 -0.8) (end 1.6 0.8) (layer "F.Fab") (width 0.1))
+    (fp_line (start -1.6 0.8) (end -1.6 -0.8) (layer "F.Fab") (width 0.1))
+    (fp_line (start -1.6 -0.8) (end 1.6 -0.8) (layer "F.Fab") (width 0.1))
+    (pad "1" smd roundrect (at -1.475 0) (size 1.15 1.8) (layers "F.Cu" "F.Paste" "F.Mask") (roundrect_rratio 0.217391)
+      (net 2 "GND") (pintype "passive"))
+    (pad "2" smd roundrect (at 1.475 0) (size 1.15 1.8) (layers "F.Cu" "F.Paste" "F.Mask") (roundrect_rratio 0.217391)
+      (net 45 "Net-(J17-Pad1)") (pintype "passive"))
+    (model "${KICAD6_3DMODEL_DIR}/Capacitor_SMD.3dshapes/C_1206_3216Metric.wrl"
+      (offset (xyz 0 0 0))
+      (scale (xyz 1 1 1))
+      (rotate (xyz 0 0 0))
     )
   )
@@
   )
   (footprint "Connector_PinHeader_2.54mm:PinHeader_1x02_P2.54mm_Vertical" (layer "F.Cu")
-    (at 113.36 115 90)
+    (at 113.125 112.4 90)
     (descr "Through hole straight pin header, 1x02, 2.54mm pitch, single row")
     (tags "Through hole pin header THT 1x02 2.54mm single row")
@@
   (segment (start 117.61 120.33) (end 119.07 120.33) (width 0.25) (layer "F.Cu") (net 43))
   (segment (start 120.4 118.1) (end 121.75 118.1) (width 0.25) (layer "F.Cu") (net 43))
-  (segment (start 112.59 120.4) (end 112.66 120.33) (width 0.25) (layer "F.Cu") (net 44))
-  (segment (start 113.36 115) (end 110.2 115) (width 0.25) (layer "F.Cu") (net 44))
-  (segment (start 110.2 120.4) (end 112.59 120.4) (width 0.25) (layer "F.Cu") (net 44))
-  (segment (start 110.2 115) (end 110.2 120.4) (width 0.25) (layer "F.Cu") (net 44))
+  (segment (start 112.66 120.33) (end 112.59 120.4) (width 0.25) (layer "F.Cu") (net 44))
+  (segment (start 112.59 120.4) (end 110.2 120.4) (width 0.25) (layer "F.Cu") (net 44))
+  (segment (start 110.2 112.4) (end 113.125 112.4) (width 0.25) (layer "F.Cu") (net 44))
+  (segment (start 110.2 120.4) (end 110.2 112.4) (width 0.25) (layer "F.Cu") (net 44))
+  (segment (start 115.86 117.94) (end 116 117.8) (width 0.25) (layer "F.Cu") (net 45))
   (segment (start 114.2 127.7) (end 115.3 127.7) (width 0.25) (layer "F.Cu") (net 45))
+  (segment (start 117.6 117.8) (end 117.675 117.725) (width 0.25) (layer "F.Cu") (net 45))
   (segment (start 116.04 119.06) (end 117.61 119.06) (width 0.25) (layer "F.Cu") (net 45))
+  (segment (start 117.675 117.725) (end 117.675 116.2) (width 0.25) (layer "F.Cu") (net 45))
   (segment (start 114.2 125.5625) (end 114.2625 125.5) (width 0.25) (layer "F.Cu") (net 45))
-  (segment (start 115.86 119.24) (end 116.04 119.06) (width 0.25) (layer "F.Cu") (net 45))
+  (segment (start 116 117.8) (end 117.6 117.8) (width 0.25) (layer "F.Cu") (net 45))
   (segment (start 114.2 129.925) (end 114.2 127.7) (width 0.25) (layer "F.Cu") (net 45))
   (segment (start 115.86 127.14) (end 115.86 119.24) (width 0.25) (layer "F.Cu") (net 45))
   (segment (start 114.2 127.7) (end 114.2 125.5625) (width 0.25) (layer "F.Cu") (net 45))
+  (segment (start 115.86 119.24) (end 115.86 117.94) (width 0.25) (layer "F.Cu") (net 45))
   (segment (start 115.3 127.7) (end 115.86 127.14) (width 0.25) (layer "F.Cu") (net 45))
   (segment (start 110.1 121.6) (end 112.66 121.6) (width 0.25) (layer "F.Cu") (net 48))

Commit message: major updates to interface, analytics and security
Parts:
- added R11: 1k, Resistor_SMD:R_1206_3216Metric, F.Cu at (120.5, 114.1)
Routing:
- net Net-(J17-Pad1): track 20.5 -> 28.0 mm
- net Net-(D7-Pad1): track 5.59 -> 8.17 mm
- net GND: vias 20 -> 12

Commit message: recent changes
Parts:
- removed J10: V Reg in, Connector_PinHeader_2.54mm:PinHeader_1x02_P2.54mm_Vertical
- removed J11, J9: V reg out, Connector_PinHeader_2.54mm:PinHeader_1x02_P2.54mm_Vertical
- removed J14: V chrg out, Connector_PinHeader_2.54mm:PinHeader_1x02_P2.54mm_Vertical
- removed J15: V Low Batt in, Connector_PinHeader_2.54mm:PinHeader_1x02_P2.54mm_Vertical
- removed J16: V ref in, Connector_PinHeader_2.54mm:PinHeader_1x02_P2.54mm_Vertical
- removed J17: V Batt in, Connector_PinHeader_2.54mm:PinHeader_1x02_P2.54mm_Vertical
- removed J18: V Low Batt out, Connector_PinHeader_2.54mm:PinHeader_1x02_P2.54mm_Vertical
- removed J7: V sys in, Connector_PinHeader_2.54mm:PinHeader_1x02_P2.54mm_Vertical
- added C14: 10uF, Capacitor_SMD:C_1206_3216Metric, F.Cu at (153.3, 98.4)
- added R12: 0, Resistor_SMD:R_1206_3216Metric, F.Cu at (115.4, 126.9)
- added R13: 0, Resistor_SMD:R_1206_3216Metric, F.Cu at (115.7, 132.3)
- added R14: 0/160, Resistor_SMD:R_1206_3216Metric, F.Cu at (147.9, 98.2)
- J8: value Cell Module -> cell data headers; footprint Connector_PinHeader_2.54mm:PinHeader_1x02_P2.54mm_Vertical -> Connector_PinSocket_2.54mm:PinSocket_1x03_P2.54mm_Vertical
- L1: footprint Inductor_SMD:L_1206_3216Metric -> Inductor_SMD:L_Bourns-SRU8028_8.0x8.0mm
- L2: footprint Inductor_SMD:L_1206_3216Metric -> Inductor_SMD:L_Bourns-SRN8040_8x8.15mm
- U4: footprint Package_SO:SOIC-8_3.9x4.9mm_P1.27mm -> Package_DIP:DIP-8_W7.62mm
- moved J6 29.7 mm to (147.8, 124.9)
- moved J1 25.1 mm to (131.6, 100.1)
- moved C6 22.3 mm to (115.7, 134.9), turned to 180 degrees
- moved R7 22.2 mm to (109.7, 108.8), turned to -90 degrees
- moved R6 14.2 mm to (114.3, 111.4)
- moved C13 7.41 mm to (118.9, 109.3), turned to 90 degrees
- moved U4 7.35 mm to (109.9, 115.8)
- moved C7 6.43 mm to (151.7, 130.6)
- moved R1 5.85 mm to (151.1, 135.8), turned to 180 degrees
- moved D3 4.98 mm to (121.0, 81.7), turned to 180 degrees
- moved R11 4.72 mm to (121.8, 109.6)
- moved J8 4.35 mm to (131.9, 119.8), turned to 180 degrees
- moved U2 2.78 mm to (125.3, 132.7)
- moved L1 2.27 mm to (137.0, 127.8), turned to 180 degrees
- moved L2 2.23 mm to (129.8, 87.4)
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Connections:
- C13 pad 2: Net-(J17-Pad1) -> Net-(C13-Pad2)
- C6 pad 1: Net-(C6-Pad1) -> Net-(C13-Pad2)
- C7 pad 1: Net-(C7-Pad1) -> VCC
- J8 pad 1: Net-(J8-Pad1) -> Net-(J6-Pad3)
- L1 pad 2: Net-(C7-Pad1) -> VCC
- R11 pad 1: Net-(J17-Pad1) -> Net-(C13-Pad2)
- R2 pad 1: Net-(C7-Pad1) -> VCC
- R6 pad 1: Net-(J17-Pad1) -> Net-(C13-Pad2)
- U1 pad 12: Net-(J8-Pad1) -> unconnected-(U1-Pad12)
- U1 pad 13: Net-(J8-Pad2) -> Net-(J8-Pad3)
- U1 pad 14: Net-(J15-Pad1) -> Net-(J8-Pad2)
- U1 pad 15: unconnected-(U1-Pad15) -> Net-(C11-Pad1)
- U1 pad 17: unconnected-(U1-Pad17) -> Net-(J6-Pad4)
- U1 pad 18: unconnected-(U1-Pad18) -> Net-(J6-Pad3)
- U1 pad 19: unconnected-(U1-Pad19) -> Net-(J6-Pad5)
- U1 pad 2: Net-(J6-Pad6) -> unconnected-(U1-Pad2)
- U1 pad 23: Net-(J1-Pad3) -> unconnected-(U1-Pad23)
- U1 pad 25: Net-(J3-Pad3) -> Net-(C14-Pad2)
- U1 pad 3: Net-(J6-Pad5) -> unconnected-(U1-Pad3)
- U1 pad 4: Net-(J6-Pad4) -> unconnected-(U1-Pad4)
- U1 pad 5: Net-(J6-Pad3) -> Net-(J1-Pad3)
- U1 pad 6: unconnected-(U1-Pad6) -> Net-(J6-Pad6)
- U2 pad 10: Net-(C6-Pad1) -> Net-(C13-Pad2)
- U4 pad 2: Net-(J16-Pad1) -> Net-(R6-Pad2)
- U4 pad 3: Net-(R6-Pad2) -> Net-(R12-Pad1)
- U4 pad 8: Net-(J17-Pad1) -> Net-(C13-Pad2)
Routing:
- net Net-(C13-Pad2): track 0.00 -> 65.3 mm, vias 0 -> 3
- net VCC: track 98.5 -> 161.0 mm
- net Net-(C10-Pad1): track 30.1 -> 74.6 mm
- net Net-(J17-Pad1): track 28.0 -> 0.00 mm
- net Net-(J6-Pad3): track 4.79 -> 29.6 mm
- net Net-(C7-Pad1): track 23.5 -> 0.00 mm
- net Net-(J6-Pad6): track 4.79 -> 23.0 mm, vias 0 -> 1
- net Net-(C11-Pad1): track 10.0 -> 26.6 mm, vias 0 -> 1
- net Net-(C14-Pad2): track 0.00 -> 14.0 mm
- net Net-(J16-Pad1): track 13.4 -> 0.00 mm
- net Net-(D6-Pad1): track 25.1 -> 36.5 mm, vias 2 -> 3
- net Net-(J1-Pad3): track 15.8 -> 5.40 mm
- net Net-(L2-Pad1): track 3.77 -> 13.7 mm, vias 0 -> 2
- net Net-(C6-Pad1): track 9.01 -> 0.00 mm
- net Net-(R12-Pad1): track 0.00 -> 8.57 mm
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